File: qsd2.kicad_sch (KiCad schematic)
At the start: 65 parts, among them J1 5-1814832-1, J2 5-1814832-1, J3 Conn_02x08_Odd_Even, J4 SJ-3524-SMT, U1 SN74LVC1G14DBV, U10 GALI-39, U2 SN74LVC1G14DBV, U3 SN74CBT3253, U4 SN74AC74PW, U5 AD8226ARZ-R7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

Commit message: Initial commit.
Parts:
- U3: footprint Package_SO:TSSOP-16_4.4x5mm_P0.65mm -> Package_SO:SOIC-16_3.9x9.9mm_P1.27mm
- U4: footprint Package_SO:TSSOP-14_4.4x5mm_P0.65mm -> Package_SO:SOIC-14_3.9x8.7mm_P1.27mm
- U5, U6: footprint 16TSOP:R_8_ADI -> AD8226:R_8_ADI
Changed lines of the file:
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@@
 			)
 		)
-		(property "Footprint" "Package_SO:TSSOP-14_4.4x5mm_P0.65mm"
+		(property "Footprint" "Package_SO:SOIC-14_3.9x8.7mm_P1.27mm"
 			(at 125.095 46.99 0)
 			(effects
@@
 			)
 		)
-		(property "Footprint" "16TSOP:R_8_ADI"
+		(property "Footprint" "AD8226:R_8_ADI"
 			(at 193.04 127.635 0)
 			(effects
@@
 			)
 		)
-		(property "Footprint" "Package_SO:TSSOP-16_4.4x5mm_P0.65mm"
+		(property "Footprint" "Package_SO:SOIC-16_3.9x9.9mm_P1.27mm"
 			(at 111.76 104.14 0)
 			(effects
@@
 			)
 		)
-		(property "Footprint" "16TSOP:R_8_ADI"
+		(property "Footprint" "AD8226:R_8_ADI"
 			(at 193.675 83.82 0)
 			(effects

Commit message: QSD2EZ to V1.0 fab.
Connections:
- net at C33.2, R15.2, R5.1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: now also TR1.2
Changed lines of the file:
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@@
 	)
 	(junction
+		(at 91.44 88.9)
+		(diameter 0)
+		(color 0 0 0 0)
+	)
+	(junction
 		(at 111.76 77.47)
 		(diameter 0)
@@
 	(wire
 		(pts
-			(xy 91.44 96.52) (xy 91.44 81.28)
+			(xy 91.44 96.52) (xy 91.44 88.9)
 		)
 		(stroke
@@
 	(wire
 		(pts
+			(xy 76.835 88.9) (xy 91.44 88.9)
+		)
+		(stroke
+			(width 0)
+			(type default)
+		)
+	)
+	(wire
+		(pts
 			(xy 102.235 49.53) (xy 107.315 49.53)
 		)
@@
 	(wire
 		(pts
+			(xy 76.835 96.52) (xy 76.835 88.9)
+		)
+		(stroke
+			(width 0)
+			(type default)
+		)
+	)
+	(wire
+		(pts
 			(xy 90.805 101.6) (xy 92.71 101.6)
 		)
@@
 	(wire
 		(pts
+			(xy 91.44 88.9) (xy 91.44 81.28)
+		)
+		(stroke
+			(width 0)
+			(type default)
+		)
+	)
+	(wire
+		(pts
 			(xy 20.955 114.935) (xy 20.955 117.475)
 		)
@@
 	(wire
 		(pts
+			(xy 80.645 96.52) (xy 76.835 96.52)
+		)
+		(stroke
+			(width 0)
+			(type default)
+		)
+	)
+	(wire
+		(pts
 			(xy 250.19 103.505) (xy 252.73 103.505)
 		)
@@
 		(pin "6"
 		)
+		(pin "2"
+		)
 		(instances

Commit message: Updated README and BOM for QSD2EZ.
Parts:
- TR1: value ADT4-6T -> ADT4-6T+
Other:
- note added: "QSD2EZ with Divide-by-Two Quadrature Double-Balanced"
- note removed: "QSD with Divide-by-Two Quadrature Double-Balanced"
- title: QSD2 with Divide-by-Two Quadrature Double-Balanced -> QSD2EZ with Divide-by-Two Quadrature Double-Balanced
Changed lines of the file:
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@@
 	(paper "A4")
 	(title_block
-		(title "QSD2 with Divide-by-Two Quadrature Double-Balanced")
-		(date "2024-02-29")
-		(rev "1.1")
+		(title "QSD2EZ with Divide-by-Two Quadrature Double-Balanced")
+		(date "2024-05-07")
+		(rev "1.0")
 	)
 	(junction
@@
 		)
 	)
-	(text "QSD with Divide-by-Two Quadrature Double-Balanced"
+	(text "QSD2EZ with Divide-by-Two Quadrature Double-Balanced"
 		(exclude_from_sim no)
 		(at 72.39 22.225 0)
@@
 			)
 		)
-		(property "Value" "ADT4-6T"
+		(property "Value" "ADT4-6T+"
 			(at 85.725 104.14 0)
 			(effects
