File: qsd2.kicad_sch (KiCad schematic)
At the start: 69 parts, among them J1 5-1814832-1, J2 5-1814832-1, J3 Conn_02x08_Odd_Even, J4 SJ-3524-SMT, J5 B4B-XH-A_LF__SN_, U1 SN74LVC1G14DBV, U10 GALI-39, U2 SN74LVC1G14DBV, U3 SN74CBT3253, U4 SN74AC74PW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

Commit message: Ready for fab QSD2EZ V1.1 May 21, 2026.
Parts:
- removed C13, C26: 1uF, Capacitor_SMD:C_1206_3216Metric, symbol Device:C_Small
- removed U7, U8: AP2120N-2.5TRG1, AP2120N:SOT-23_DIO, symbol 2023-10-04_14-49-55:AP2120N-2.5TRG1
- added C8: 0.1uF, Capacitor_SMD:C_1206_3216Metric, symbol Device:C_Small
- added R18, R19: 4.7k, Resistor_SMD:R_1206_3216Metric, symbol Device:R_Small_US
- added TP3: TestPoint, Connector_PinHeader_2.54mm:PinHeader_1x01_P2.54mm_Vertical, symbol Connector:TestPoint
- added U11: SN74LVC1G14DBV, Package_TO_SOT_SMD:SOT-23-5, symbol 74xGxx:SN74LVC1G14DBV
- added U12, U13: LM4040DBZ-2.5, Package_TO_SOT_SMD:SOT-23, symbol Reference_Voltage:LM4040DBZ-2.5
Connections:
- net 5V_FILT: now also C8.2, R18.2, R19.2, U11.5 (VCC)
- net CLK1: now also U2.4, U11.2; no longer J1.2, U2.2
- net CLK2: now also U11.4; no longer U2.4
- net GND: now also C8.1, TP3.1, U11.3 (GND), U12.2 (A), U13.2 (A)
- net REF_I: now also R18.1, U12.1 (K)
- net REF_Q: now also R19.1, U13.1 (K)
- new net: J1.2, U2.2
Other:
- note added: "2.5V REFERENCE"
- note added: "This is a grounded header pin for attaching a probe."
- moved on the sheet: C1, C22, C23, C27, C31, R28, TP1, TP2, U1, U4
